File: PCB/0_10v_driver.kicad_sch (KiCad schematic)
At the start: 0 parts

Commit message: fix to 0-10V IN schematic, 0-10V OUT schematic
Parts:
- added C4: 16V 1uF X7R ±5% 0603, Capacitor_SMD:C_0603_1608Metric_Pad1.08x0.95mm_HandSolder, symbol Device:C
- added C5: 100nF 50V X7R ±5% 0603, Capacitor_SMD:C_0603_1608Metric_Pad1.08x0.95mm_HandSolder, symbol Device:C
- added D1: SR70, SamacSys_Parts:SR70, symbol SamacSys_Parts:SR70
- added D4: CDSOD323-T15, SamacSys_Parts:CDSOD323T15, symbol SamacSys_Parts:CDSOD323-T15
- added IC1: GP8403-TC50-EW, SamacSys_Parts:SOP100P600X165-11N, symbol SamacSys_Parts:GP8403-TC50-EW
- added J2: Conn_01x02_Socket, symbol Connector:Conn_01x02_Socket
- added NT2: NetTie_2, symbol Device:NetTie_2
- added R6, R7, R8: 0R 5% 0402 1/16W, Resistor_SMD:R_0402_1005Metric_Pad0.72x0.64mm_HandSolder, symbol Device:R
Connections:
- new net: C5.1, D1.2 (I/O_1), D4.1 (K), IC1.8 (VOUT0)
- new net: D1.3 (I/O_2), J2.2 (Pin_2)
- new net: IC1.3 (A0), R6.2
- new net: C4.1, IC1.10 (V5V)
- new net: IC1.4 (A1), R7.2
- new net: IC1.9 (A2), R8.1
- new net GND: C4.2, D1.1 (GND), D4.2 (A), IC1.11 (EP), NT2.2, R6.1, R7.1, R8.2
- new net GNDA_2: C5.2, IC1.6 (GND), J2.1 (Pin_1), NT2.1
- new net SCLK: IC1.1 (SCLK)
- new net SDA: IC1.2 (SDA)
- new net VCC: D1.4 (VCC), IC1.5 (VCC)
- no-connect marks 0 -> 1
Other:
- note added: "Datasheet https://dfimg.dfrobot.com/nobody/wiki/79daa2f3c729e78f0580b474fe33a5e3.pdf https://jlcpcb.com/api/file/downloadByFileSystemAccessId/8589834510297960448"
- note added: "PULL UP i2c su ESP"
- note added: "“The GP8403 I²C address selection pins A0, A1 and A2 are hard-strapped to GND. Address configuration is fixed and not user-accessible, ensuring deterministic I²C behaviour and eliminating floating address risks.”"

Commit message: fix to 0-10v out.... idiot me :(
Connections:
- net at C5.1, D1.2 (I/O_1), D4.1 (K)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: now also J2.2 (Pin_2)
- net at D1.3 (I/O_2): no longer J2.2 (Pin_2)
- no-connect marks 1 -> 2
Other:
- note added: "questo è per due linee non va bene... a meno che non si voglia prevedere secondo 0-10V output."
Changed lines of the file:
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@@
+		)
+	)
+	(text "questo è per due linee non va bene...\na meno che non si voglia prevedere secondo 0-10V output. \n"
+		(exclude_from_sim no)
+		(at 184.15 71.628 0)
+		(effects
+			(font
+				(size 1.27 1.27)
+				(color 255 0 40 1)
+			)
 		)
 	)
@@
 	)
 	(junction
+		(at 166.37 78.74)
+		(diameter 0)
+		(color 0 0 0 0)
+	)
+	(junction
 		(at 152.4 78.74)
 		(diameter 0)
@@
 		(diameter 0)
 		(color 0 0 0 0)
+	)
+	(no_connect
+		(at 196.85 78.74)
 	)
 	(no_connect
@@
 	(wire
 		(pts
+			(xy 209.55 78.74) (xy 209.55 67.31)
+		)
+		(stroke
+			(width 0)
+			(type default)
+		)
+	)
+	(wire
+		(pts
 			(xy 166.37 96.52) (xy 166.37 81.28)
 		)
@@
 	(wire
 		(pts
+			(xy 166.37 67.31) (xy 166.37 78.74)
+		)
+		(stroke
+			(width 0)
+			(type default)
+		)
+	)
+	(wire
+		(pts
 			(xy 77.47 81.28) (xy 82.55 81.28)
 		)
@@
 	(wire
 		(pts
+			(xy 209.55 67.31) (xy 166.37 67.31)
+		)
+		(stroke
+			(width 0)
+			(type default)
+		)
+	)
+	(wire
+		(pts
 			(xy 152.4 96.52) (xy 152.4 93.98)
 		)
@@
 		)
 		(stroke
-			(width 0)
-			(type default)
-		)
-	)
-	(wire
-		(pts
-			(xy 196.85 78.74) (xy 209.55 78.74)
-		)
-		(stroke

Commit message: minor fix, esp32 partial schematic
Parts:
- added C6: 1uF 50V X7R ±10% 0603, Capacitor_SMD:C_0603_1608Metric_Pad1.08x0.95mm_HandSolder, symbol Device:C
- added C7: 100nF 50V X7R ±5% 0603, Capacitor_SMD:C_0603_1608Metric_Pad1.08x0.95mm_HandSolder, symbol Device:C
- added R9: 330R 0.1% 0603 1/10W, symbol Device:R
- C4: value 16V 1uF X7R ±5% 0603 -> 1uF 50V X7R ±10% 0603; MPN CC0603JRX7R7BB105 -> CC0603KRX7R9BB105
Connections:
- net GND: now also C4.1, C6.2, C7.2; no longer C4.2
- net VCC: now also C4.2, C7.1; no longer D1.4 (VCC)
- net at C5.1, D1.2 (I/O_1), D4.1 (K)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: now also R9.2; no longer IC1.8 (VOUT0)
- net at IC1.10 (V5V): now also C6.1; no longer C4.1
- new net: IC1.8 (VOUT0), R9.1
- no-connect marks 2 -> 3
Other:
- note added: "preverdere ESD si gle line to GND al posto di sr70."
- note removed: "questo è per due linee non va bene... a meno che non si voglia prevedere secondo 0-10V output."
- moved on the sheet: C5, R8

Commit message: esp32 various fix, 20to3v3 DCDC.
Parts:
- NT2: footprint (none) -> Jumper:SolderJumper-2_P1.3mm_Bridged_Pad1.0x1.5mm
- R9: footprint (none) -> Resistor_SMD:R_0603_1608Metric_Pad0.98x0.95mm_HandSolder
Connections:
- net SCLK renamed SCL
Other:
- note added: "preverdere ESD single line to GND al posto di sr70."
- note removed: "preverdere ESD si gle line to GND al posto di sr70."
Changed lines of the file:
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@@
 		)
 	)
-	(text "preverdere ESD si gle line to GND al posto di sr70."
+	(text "preverdere ESD single line to GND al posto di sr70."
 		(exclude_from_sim no)
 		(at 184.15 71.628 0)
@@
 		)
 	)
-	(hierarchical_label "SCLK"
+	(hierarchical_label "SCL"
 		(shape input)
 		(at 43.18 73.66 180)
@@
 			)
 		)
-		(property "Footprint" ""
+		(property "Footprint" "Resistor_SMD:R_0603_1608Metric_Pad0.98x0.95mm_HandSolder"
 			(at 132.08 80.518 90)
 			(effects
@@
 			)
 		)
-		(property "Footprint" ""
+		(property "Footprint" "Jumper:SolderJumper-2_P1.3mm_Bridged_Pad1.0x1.5mm"
 			(at 142.24 111.76 0)
 			(effects
