File: PCB/0_10v_input.kicad_sch (KiCad schematic)
At the start: 12 parts, among them IC2 TLV9061IDBVR, J1 Conn_01x02_Socket

Commit message: fix to 0-10V IN schematic, 0-10V OUT schematic
Parts:
- added D3: SR70, SamacSys_Parts:SR70, symbol SamacSys_Parts:SR70
- IC2: footprint SOT95P280X145-5N -> SamacSys_Parts:SOT95P280X145-5N
Connections:
- net GND: now also D2.2 (A), D3.1 (GND)
- net GNDA: no longer D2.2 (A)
- net at D2.1 (K), R1.1: now also D3.3 (I/O_2); no longer J1.2 (Pin_2)
- new net: D3.2 (I/O_1), J1.2 (Pin_2)
- no-connect marks 0 -> 1
Other:
- note added: "non va bene vcc float. serve esd diode con clamp singolo a gnd. trovare alternativa"
- note removed: "Quetsto è un po' costoso."
- moved on the sheet: D2, J1, R1

Commit message: minor fix, esp32 partial schematic
Parts:
- C2: value 100nF 16V X7R ±5% 0603 -> 100nF 50V X7R ±5% 0603; MPN CC0603JRX7R7BB104 -> CC0603JRX7R9BB104
- C3: value 16V 1uF X7R ±5% 0603 -> 1uF 50V X7R ±10% 0603; MPN CC0603JRX7R7BB105 -> CC0603KRX7R9BB105
Connections:
- net +3V3: now also C3.2; no longer C3.1
- net GNDA: now also C3.1; no longer C3.2
- net at D2.1 (K), R1.1: now also D3.2 (I/O_1), J1.2 (Pin_2); no longer D3.3 (I/O_2)
- no-connect marks 1 -> 2
Other:
- note added: "preverdere ESD si gle line to GND al posto di sr70."
- note removed: "non va bene vcc float. serve esd diode con clamp singolo a gnd. trovare alternativa"
- moved on the sheet: D3

Commit message: esp32 various fix, 20to3v3 DCDC.
Parts:
- added C13: 100nF 50V X7R ±5% 0603, Capacitor_SMD:C_0603_1608Metric_Pad1.08x0.95mm_HandSolder, symbol Device:C
- NT1: footprint (none) -> Jumper:SolderJumper-2_P1.3mm_Bridged_Pad1.0x1.5mm
Connections:
- net V_SENSE_OUT: now also C13.1
- net GNDA renamed GNDA_1
- net GNDA_1: now also C13.2
Other:
- note added: "Occhio che produce una fcut a 1,6Hz e un delay di 0.1s. Lo voglio veramente?"
- note added: "Suggested by https://documentation.espressif.com/projects/esp-hardware-design-guidelines/en/latest/esp32c6/schematic-checklist.html?title=ESP32-C6%20Hardware%20Design%20Guidelines in ADC section"
Changed lines of the file:
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@@
 	(generator_version "9.0")
 	(paper "A4")
+	(rectangle
+		(start 223.52 90.17)
+		(end 267.97 110.49)
+		(stroke
+			(width 0)
+			(type default)
+		)
+		(fill
+			(type none)
+		)
+	)
 	(text "Rilevamento linea 0-10 V non presente - Alternative e scelta progettuale\n\nIl rilevamento della presenza della linea di comando 0-10 V può essere implementato con diverse strategie, ciascuna con specifici compromessi tra semplicità hardware, affidabilità e robustezza di sistema.\n\n1) Pull-down passivo (fail-safe)- AMBIGUO\nL'aggiunta di un resistore ad alto valore verso GND (tipicamente ~1 MΩ) forza la linea a 0 V in caso di linea aperta.\nQuesta soluzione è semplice e robusta e garantisce un comportamento fail-safe (open line → 0%), ma non consente di distinguere in modo certo tra una linea realmente a 0 V e una linea scollegata.\n\n2) Bias fisso della linea - possibilità!\nLa linea viene polarizzata verso un valore intermedio o definito tramite resistori ad alta impedenza. In caso di linea aperta, il nodo assume un valore \"non valido\" riconoscibile via firmware.\nQuesta tecnica permette il rilevamento hardware dell'open line, ma può influenzare sorgenti 0-10 V esterne e introduce ambiguità in presenza di driver con pull-up interni.\n\n3) Misura di impedenza / corrente - difficile\nLa presenza della linea viene dedotta iniettando una corrente nota o misurando l'impedenza del nodo. È una soluzione robusta e industriale, ma richiede hardware aggiuntivo e maggiore complessità di validazione.\n\n4) Pull-down + test attivo con weak pull-up (soluzione adottata)\nLa linea è mantenuta fail-safe tramite un pull-down ad alta impedenza. Periodicamente, il firmware abilita per un tempo limitato un pull-up molto debole (tramite GPIO e resistore nell'ordine dei MΩ).\nSe la tensione sul nodo varia in modo misurabile, la linea è da considerarsi scollegata o ad alta impedenza; se rimane stabile, la linea è pilotata da una sorgente esterna.\nSe abilito un weak pull-up per un breve intervallo e NON vedo una variazione significativa di tensione (ΔV) entro un tempo ΔT, allora la linea 0-10 V è pilotata da una sorgente esterna ed è quindi collegata.\n\nQuesta soluzione rappresenta il miglior compromesso perché:\n\nmantiene un comportamento sicuro e prevedibile in condizioni normali;\n\nnon influenza il funzionamento dei driver 0-10 V esterni;\n\nconsente una distinzione affidabile tra \"0 V reale\" e \"linea non presente\";\n\nintroduce complessità minima e nessun impatto EMC significativo.\n\nPer questi motivi, il rilevamento tramite test attivo con weak pull-up è considerato la scelta più robusta e flessibile per applicazioni 0-10 V in ambito lighting e building control."
 		(exclude_from_sim no)
@@
 			)
 			(justify left)
+		)
+	)
+	(text "Occhio che produce una fcut a 1,6Hz e un delay di 0.1s. Lo voglio veramente?"
+		(exclude_from_sim no)
+		(at 270.002 101.854 0)
+		(effects
+			(font
+				(size 1.27 1.27)
+				(thickness 0.254)
+				(bold yes)
+			)
+		)
+	)
+	(text "Suggested by https://documentation.espressif.com/projects/esp-hardware-design-guidelines/en/latest/esp32c6/schematic-checklist.html?title=ESP32-C6%20Hardware%20Design%20Guidelines in ADC section"
+		(exclude_from_sim no)
+		(at 334.01 99.314 0)
+		(effects
+			(font
+				(size 1.27 1.27)
+				(thickness 0.254)
+				(bold yes)
+			)
 		)
 	)
@@
 	)
 	(junction
+		(at 229.87 86.36)
+		(diameter 0)
+		(color 0 0 0 0)
+	)
+	(junction
 		(at 185.42 88.9)
 		(diameter 0)
@@
 	(wire
 		(pts
-			(xy 223.52 86.36) (xy 234.95 86.36)
+			(xy 223.52 86.36) (xy 229.87 86.36)
 		)
 		(stroke
@@
 	(wire
 		(pts
+			(xy 229.87 91.44) (xy 229.87 86.36)
+		)
+		(stroke
+			(width 0)
+			(type default)
+		)
+	)
+	(wire
+		(pts
 			(xy 113.03 81.28) (xy 119.38 81.28)
 		)
@@
 	(wire
 		(pts
+			(xy 229.87 86.36) (xy 234.95 86.36)
+		)
+		(stroke
+			(width 0)
+			(type default)
+		)
+	)
+	(wire
+		(pts
 			(xy 187.96 86.36) (xy 196.85 86.36)
 		)
@@
 		(pts
 			(xy 132.08 91.44) (xy 158.75 91.44)
+		)
+		(stroke
+			(width 0)
+			(type default)
+		)
+	)
+	(wire
+		(pts
+			(xy 229.87 102.87) (xy 229.87 99.06)
 		)
 		(stroke
@@
 			)
 		)
-		(property "Value" "GNDA"
+		(property "Value" "GNDA_1"
 			(at 185.42 107.95 0)
 			(effects
@@
 			)
 		)
-		(property "Value" "GNDA"
+		(property "Value" "GNDA_1"
 			(at 193.04 107.95 0)
 			(effects
@@
 				(path "/6bd10cb8-11ca-4919-a8d8-88b44cd4cac7/8cfa68d9-1d86-47fe-9b0a-5b7093a7a1de"
 					(reference "#PWR010")
+					(unit 1)
+				)
+			)
+		)
+	)
+	(symbol
+		(lib_id "Device:C")
+		(at 229.87 95.25 0)
+		(unit 1)
+		(exclude_from_sim no)
+		(in_bom yes)
+		(on_board yes)
+		(dnp no)
+		(fields_autoplaced yes)
+		(property "Reference" "C13"
+			(at 233.68 93.9799 0)
+			(effects
+				(font
+					(size 1.27 1.27)
+				)
+				(justify left)
+			)
+		)
+		(property "Value" "100nF 50V X7R ±5% 0603"
+			(at 233.68 96.5199 0)
+			(effects
+				(font
+					(size 1.27 1.27)
+				)
+				(justify left)
+			)
+		)
+		(property "Footprint" "Capacitor_SMD:C_0603_1608Metric_Pad1.08x0.95mm_HandSolder"
+			(at 230.8352 99.06 0)
+			(effects
+				(font
+					(size 1.27 1.27)
+				)
+				(hide yes)
+			)
+		)
+		(property "Datasheet" "~"
+			(at 229.87 95.25 0)
+			(effects
+				(font
+					(size 1.27 1.27)
+				)
+				(hide yes)
+			)
+		)
+		(property "Description" "Unpolarized capacitor"
+			(at 229.87 95.25 0)
+			(effects
+				(font
+					(size 1.27 1.27)
+				)
+				(hide yes)
+			)
+		)
+		(property "MPN" "CC0603JRX7R9BB104"
+			(at 229.87 95.25 0)
+			(effects
+				(font
+					(size 1.27 1.27)
+				)
+				(hide yes)
+			)
+		)
+		(property "Manifacturer" "YAGEO"
+			(at 229.87 95.25 0)
+			(effects
+				(font
+					(size 1.27 1.27)
+				)
+				(hide yes)
+			)
+		)
+		(pin "1"
+		)
+		(pin "2"
+		)
+		(instances
+			(project "PCB"
+				(path "/6bd10cb8-11ca-4919-a8d8-88b44cd4cac7/8cfa68d9-1d86-47fe-9b0a-5b7093a7a1de"
+					(reference "C13")
 					(unit 1)
 				)
@@
 			)
 		)
-		(property "Value" "GNDA"
+		(property "Value" "GNDA_1"
 			(at 135.89 120.6499 90)
 			(effects
@@
 			)
 		)
-		(property "Value" "GNDA"
+		(property "Value" "GNDA_1"
 			(at 41.91 91.44 0)
 			(effects
@@
 			)
 		)
-		(property "Value" "GNDA"
+		(property "Value" "GNDA_1"
 			(at 119.38 106.68 0)
 			(effects
@@
 			)
 		)
-		(property "Value" "GNDA"
+		(property "Value" "GNDA_1"
 			(at 132.08 106.68 0)
 			(effects
@@
 			)
 		)
-		(property "Value" "GNDA"
+		(property "Value" "GNDA_1"
 			(at 154.94 106.68 0)
 			(effects
@@
 	)
 	(symbol
+		(lib_id "power:GNDA")
+		(at 229.87 102.87 0)
+		(unit 1)
+		(exclude_from_sim no)
+		(in_bom yes)
+		(on_board yes)
+		(dnp no)
+		(fields_autoplaced yes)
+		(property "Reference" "#PWR043"
+			(at 229.87 109.22 0)
+			(effects
+				(font
+					(size 1.27 1.27)
+				)
+				(hide yes)
+			)
+		)
+		(property "Value" "GNDA_1"
+			(at 229.87 107.95 0)
+			(effects
+				(font
+					(size 1.27 1.27)
+				)
+			)
+		)
+		(property "Footprint" ""
+			(at 229.87 102.87 0)
+			(effects
+				(font
+					(size 1.27 1.27)
+				)
+				(hide yes)
+			)
+		)
+		(property "Datasheet" ""
+			(at 229.87 102.87 0)
+			(effects
+				(font
+					(size 1.27 1.27)
+				)
+				(hide yes)
+			)
+		)
+		(property "Description" "Power symbol creates a global label with name \"GNDA\" , analog ground"
+			(at 229.87 102.87 0)
+			(effects
+				(font
+					(size 1.27 1.27)
+				)
+				(hide yes)
+			)
+		)
+		(pin "1"
+		)
+		(instances
+			(project "PCB"
+				(path "/6bd10cb8-11ca-4919-a8d8-88b44cd4cac7/8cfa68d9-1d86-47fe-9b0a-5b7093a7a1de"
+					(reference "#PWR043")
+					(unit 1)
+				)
+			)
+		)
+	)
+	(symbol
 		(lib_id "Connector:Conn_01x02_Socket")
 		(at 36.83 83.82 180)
@@
 			)
 		)
-		(property "Footprint" ""
+		(property "Footprint" "Jumper:SolderJumper-2_P1.3mm_Bridged_Pad1.0x1.5mm"
 			(at 142.24 120.65 0)
 			(effects
