File: PCB/PCB.kicad_pcb (KiCad board)
At the start: 4 copper layers, 60 x 60 mm, 37 parts, among them IC1 GP8403-TC50-EW, IC2 TLV9061IDBVR, IC3 BC847BDW1T1G, J3 BM06B-GHS-TBT_LF__SN_, U1 ESP32-C6-WROOM-1-N8, U2 ESD7004MUTAG

Commit message: stusb schematic
Parts:
- removed the C2 at (153.5, 84.2)
- removed the C2 at (112.1, 63.8)
- removed the C3 at (153.5, 86.7)
- removed the C3 at (112.1, 66.3)
- added C11: 100nF 50V X7R ±5% 0603, Capacitor_SMD:C_0603_1608Metric_Pad1.08x0.95mm_HandSolder, F.Cu at (39.8, 36.3)
- added C12: 1uF 50V X7R ±10% 0603, Capacitor_SMD:C_0603_1608Metric_Pad1.08x0.95mm_HandSolder, F.Cu at (39.8, 38.9)
- added C13: 100nF 50V X7R ±5% 0603, Capacitor_SMD:C_0603_1608Metric_Pad1.08x0.95mm_HandSolder, F.Cu at (56.7, 27.0)
- added C14: 4u7 50V 0805 X7R, Capacitor_SMD:C_0805_2012Metric_Pad1.18x1.45mm_HandSolder, F.Cu at (59.4, 55.6)
- added C15: 22pF 50V C0G 0402, Capacitor_SMD:C_0402_1005Metric_Pad0.74x0.62mm_HandSolder, F.Cu at (55.3, 55.0)
- added C16: 22uF 0805 10V X7R, Capacitor_SMD:C_0805_2012Metric_Pad1.18x1.45mm_HandSolder, F.Cu at (59.4, 58.6)
- added C17: 100nF 50V X7R 0402, Capacitor_SMD:C_0402_1005Metric_Pad0.74x0.62mm_HandSolder, F.Cu at (55.3, 57.0)
- added C18: 22uF 0805 10V X7R, Capacitor_SMD:C_0805_2012Metric_Pad1.18x1.45mm_HandSolder, F.Cu at (59.4, 61.6)
- added C19: 1uF 10V X7R 0402, Capacitor_SMD:C_0402_1005Metric_Pad0.74x0.62mm_HandSolder, F.Cu at (31.6, 61.0)
- added C2: 100nF 50V X7R ±5% 0603, Capacitor_SMD:C_0603_1608Metric_Pad1.08x0.95mm_HandSolder, F.Cu at (56.7, 22.0)
- added C20: 1uF 10V X7R 0402, Capacitor_SMD:C_0402_1005Metric_Pad0.74x0.62mm_HandSolder, F.Cu at (31.6, 63.0)
- added C21: 4u7 50V 0805 X7R, Capacitor_SMD:C_0805_2012Metric_Pad1.18x1.45mm_HandSolder, F.Cu at (30.5, 67.0)
- added C3: 1uF 50V X7R ±10% 0603, Capacitor_SMD:C_0603_1608Metric_Pad1.08x0.95mm_HandSolder, F.Cu at (56.7, 24.5)
- added D5: LED GREEN, Diode_SMD:D_0603_1608Metric_Pad1.05x0.95mm_HandSolder, F.Cu at (19.1, 47.3)
- added D6: LED BLUE, Diode_SMD:D_0603_1608Metric_Pad1.05x0.95mm_HandSolder, F.Cu at (19.1, 49.8)
- added D7: ESDA25P35-1U1M, SamacSys_Parts:ESDA25P351U1M, F.Cu at (25.6, 67.6)
- added FB2: 330Ohm@100MHz 0805, SamacSys_Parts:INDC2012X105N, F.Cu at (28.0, 47.5)
- added IC4: MPM3510AGQV, SamacSys_Parts:QFN-19, F.Cu at (65.4, 58.4)
- added J4: G-Switch GT-USB-7075A, USB_C:G-Switch GT-USB-7075A, F.Cu at (23.4, 60.8)
- added NT1: NetTie_2, Jumper:SolderJumper-2_P1.3mm_Bridged_Pad1.0x1.5mm, F.Cu at (61.1, 35.7)
- added NT2: NetTie_2, Jumper:SolderJumper-2_P1.3mm_Bridged_Pad1.0x1.5mm, F.Cu at (47.8, 66.8)
- added NT3: NetTie_2, Jumper:SolderJumper-2_P1.3mm_Bridged_Pad1.0x1.5mm, F.Cu at (63.9, 64.2)
- added R10: 10K 5% 0603 1/10W, Resistor_SMD:R_0603_1608Metric_Pad0.98x0.95mm_HandSolder, F.Cu at (44.1, 28.8)
- added R11: 3K3 1% 0603 1/10W, Resistor_SMD:R_0603_1608Metric_Pad0.98x0.95mm_HandSolder, F.Cu at (44.1, 31.3)
- added R14: 3K3 1% 0603 1/10W, Resistor_SMD:R_0603_1608Metric_Pad0.98x0.95mm_HandSolder, F.Cu at (44.1, 33.8)
- added R19: 3K3 1% 0603 1/10W, Resistor_SMD:R_0603_1608Metric_Pad0.98x0.95mm_HandSolder, F.Cu at (44.1, 36.3)
- added R21: 330R 1% 0603, Resistor_SMD:R_0603_1608Metric_Pad0.98x0.95mm_HandSolder, F.Cu at (48.5, 28.8)
- added R22: 3K3 1% 0603 1/10W, Resistor_SMD:R_0603_1608Metric_Pad0.98x0.95mm_HandSolder, F.Cu at (48.5, 31.3)
- added R23: 220R 1% 0603, Resistor_SMD:R_0603_1608Metric_Pad0.98x0.95mm_HandSolder, F.Cu at (48.5, 33.8)
- added R24: 10K 1% 0402 1/16W, Resistor_SMD:R_0402_1005Metric_Pad0.72x0.64mm_HandSolder, F.Cu at (58.6, 64.1)
- added R25: 75K 0402 1% 62.5mW, Capacitor_SMD:C_0402_1005Metric_Pad0.74x0.62mm_HandSolder, F.Cu at (55.3, 59.0)
- added R26: 24K 0402 1% 62.5mW, Capacitor_SMD:C_0402_1005Metric_Pad0.74x0.62mm_HandSolder, F.Cu at (55.3, 60.9)
- added R27: 1M 0402 5% 62.5mW, Capacitor_SMD:C_0402_1005Metric_Pad0.74x0.62mm_HandSolder, F.Cu at (55.3, 62.9)
- added R28: 10K 1% 0402 1/16W, Resistor_SMD:R_0402_1005Metric_Pad0.72x0.64mm_HandSolder, F.Cu at (31.6, 55.0)
- added R29: 10K 1% 0402 1/16W, Resistor_SMD:R_0402_1005Metric_Pad0.72x0.64mm_HandSolder, F.Cu at (31.6, 57.0)
- added R30: 10K 1% 0402 1/16W, Resistor_SMD:R_0402_1005Metric_Pad0.72x0.64mm_HandSolder, F.Cu at (31.6, 59.0)
- added R9: 330R 0.1% 0603 1/10W, Resistor_SMD:R_0603_1608Metric_Pad0.98x0.95mm_HandSolder, F.Cu at (37.4, 65.3)
- added S1: KSC221JLFS, SamacSys_Parts:KSC221JLFS, F.Cu at (46.7, 44.8)
- added U3: STUSB4500QTR, Package_DFN_QFN:QFN-24-1EP_4x4mm_P0.5mm_EP2.7x2.7mm, F.Cu at (20.0, 68.7)
- R20: value 100R 1% 0402 1/16W -> 10K 5% 0603 1/10W; footprint Resistor_SMD:R_0402_1005Metric_Pad0.72x0.64mm_HandSolder -> Resistor_SMD:R_0603_1608Metric_Pad0.98x0.95mm_HandSolder
- moved IC3 147.0 mm to (23.5, 47.8)
- moved R12 128.0 mm to (39.2, 41.1)
- moved R13 128.0 mm to (39.2, 43.1)
- moved R15 128.0 mm to (39.2, 45.1)
- moved R16 128.0 mm to (39.2, 47.1)
- moved R17 128.0 mm to (39.2, 49.1)
- moved R18 128.0 mm to (39.2, 51.1)
- moved R20 127.9 mm to (44.1, 38.9)
- moved U2 127.0 mm to (27.6, 50.2), turned to 0 degrees
- moved J3 120.2 mm to (44.6, 23.5)
- moved U1 115.4 mm to (27.2, 34.9)
- moved C10 112.9 mm to (39.8, 33.8)
- moved C8 112.9 mm to (39.8, 28.8)
- moved C9 112.9 mm to (39.8, 31.3)
- moved D3 107.9 mm to (61.9, 21.6)
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Connections:
- net GNDA renamed GNDA_1
- C8 pad 1: +3V3 -> +3V3_ESP
- C9 pad 1: +3V3 -> +3V3_ESP
- R20 pad 1: unconnected-(R20-Pad1) -> /MCU/GPIO4
- R20 pad 2: unconnected-(R20-Pad2) -> +3V3
- U1 pad 2: +3V3 -> +3V3_ESP
Other:
- board text added: "REMEMBER TO ADD ROHS TO LAYOUT (FROM JLC?)"
