File: PCB/PCB.kicad_sch (KiCad schematic)
At the start: 70 parts, among them IC1 GP8403-TC50-EW, IC2 GP8403-TC50-EW, IC3 TPS25947, Q1 STL6P3LLH6, Q2 STL6P3LLH6, Q3 STL6P3LLH6, Q4 STL6P3LLH6, U1 ESP32-C6-WROOM-1, U2 STUSB4500QTR, U3 STUSB4500QTR

Commit message: 0-10V IN schematic
Parts:
- removed IC1, IC2: GP8403-TC50-EW, SOP100P600X165-11N, symbol SamacSys_Parts:GP8403-TC50-EW
- removed IC3: TPS25947, TPS25947, symbol SamacSys_Parts:TPS25947
- removed Q1, Q2, Q3, Q4: STL6P3LLH6, STL8N10F7, symbol SamacSys_Parts:STL6P3LLH6
- removed R1, R10, R11, R12, R13, R14, R15, R16, R17, R18, R19, R2, R20, R21, R22, R23, R24, R25, R26, R27, R28, R29, R3, R30, R31, R32, R33, R34, R35, R36, R37, R38, R39, R4, R40, R41, R42, R43, R44, R45, R46, R47, R48, R49, R5, R50, R51, R52, R53, R54, R55, R56, R57, R58, R59, R6, R60, R7, R8, R9: RC0603FR-07100KL, RESC1608X55N, symbol SamacSys_Parts:RC0603FR-07100KL
- removed U1: ESP32-C6-WROOM-1, PCM_Espressif:ESP32-C6-WROOM-1, symbol PCM_Espressif:ESP32-C6-WROOM-1
- removed U2, U3: STUSB4500QTR, Package_DFN_QFN:QFN-24-1EP_4x4mm_P0.5mm_EP2.7x2.7mm, symbol Interface_USB:STUSB4500QTR
Other:
- added sheet 0-10V Input (0_10v_input.kicad_sch)

Commit message: minor fix, esp32 partial schematic
Other:
- sheet 0-10V Driver ports: added SCLK, SDA, VCC; removed none
Changed lines of the file:
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@@
+			)
+		)
+		(pin "SCLK" input
+			(at 156.21 100.33 180)
+			(effects
+				(font
+					(size 1.27 1.27)
+				)
+				(justify left)
+			)
+		)
+		(pin "SDA" bidirectional
+			(at 156.21 102.87 180)
+			(effects
+				(font
+					(size 1.27 1.27)
+				)
+				(justify left)
+			)
+		)
+		(pin "VCC" input
+			(at 166.37 96.52 90)
+			(effects
+				(font
+					(size 1.27 1.27)
+				)
+				(justify right)
 			)
 		)
@@
 	)
 	(sheet
-		(at 86.36 93.98)
-		(size 22.86 15.24)
+		(at 86.36 96.52)
+		(size 22.86 12.7)
 		(exclude_from_sim no)
 		(in_bom yes)
@@
 		)
 		(property "Sheetname" "0-10V Input"
-			(at 86.36 93.2684 0)
+			(at 86.36 95.8084 0)
 			(effects
 				(font

Commit message: esp32 various fix, 20to3v3 DCDC.
Other:
- sheet 0-10V Driver ports: added SCL; removed SCLK
- sheet DCDC_stage ports: added PG_OUT, VIN, VOUT_3V3; removed none
- sheet MCU ports: added PG_IN, SCL, SDA, V_SENSE_IN; removed none
Changed lines of the file:
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@@
 	(generator_version "9.0")
 	(paper "A4")
+	(wire
+		(pts
+			(xy 127 83.82) (xy 127 96.52)
+		)
+		(stroke
+			(width 0)
+			(type default)
+		)
+	)
+	(wire
+		(pts
+			(xy 156.21 104.14) (xy 144.78 104.14)
+		)
+		(stroke
+			(width 0)
+			(type default)
+		)
+	)
+	(wire
+		(pts
+			(xy 144.78 106.68) (xy 156.21 106.68)
+		)
+		(stroke
+			(width 0)
+			(type default)
+		)
+	)
+	(wire
+		(pts
+			(xy 109.22 106.68) (xy 119.38 106.68)
+		)
+		(stroke
+			(width 0)
+			(type default)
+		)
+	)
 	(sheet
 		(at 156.21 96.52)
@@
 			)
 		)
-		(pin "SCLK" input
-			(at 156.21 100.33 180)
+		(pin "SCL" input
+			(at 156.21 104.14 180)
 			(effects
 				(font
@@
 		)
 		(pin "SDA" bidirectional
-			(at 156.21 102.87 180)
+			(at 156.21 106.68 180)
 			(effects
 				(font
@@
 		)
 		(pin "VCC" input
-			(at 166.37 96.52 90)
+			(at 171.45 96.52 90)
 			(effects
 				(font
@@
 			)
 		)
+		(pin "PG_OUT" output
+			(at 127 83.82 270)
+			(effects
+				(font
+					(size 1.27 1.27)
+				)
+				(justify left)
+			)
+		)
+		(pin "VIN" input
+			(at 140.97 72.39 90)
+			(effects
+				(font
+					(size 1.27 1.27)
+				)
+				(justify right)
+			)
+		)
+		(pin "VOUT_3V3" output
+			(at 124.46 83.82 270)
+			(effects
+				(font
+					(size 1.27 1.27)
+				)
+				(justify left)
+			)
+		)
 		(instances
 			(project "PCB"
@@
 			)
 		)
+		(pin "SCL" output
+			(at 144.78 104.14 0)
+			(effects
+				(font
+					(size 1.27 1.27)
+				)
+				(justify right)
+			)
+		)
+		(pin "SDA" bidirectional
+			(at 144.78 106.68 0)
+			(effects
+				(font
+					(size 1.27 1.27)
+				)
+				(justify right)
+			)
+		)
+		(pin "V_SENSE_IN" input
+			(at 119.38 106.68 180)
+			(effects
+				(font
+					(size 1.27 1.27)
+				)
+				(justify left)
+			)
+		)
+		(pin "PG_IN" input
+			(at 127 96.52 90)
+			(effects
+				(font
+					(size 1.27 1.27)
+				)
+				(justify right)
+			)
+		)
 		(instances
 			(project "PCB"
@@
 		)
 		(pin "V_SENSE_OUT" output
-			(at 109.22 101.6 0)
-			(effects
-				(font
+			(at 109.22 106.68 0)
+			(effects
+				(font

Commit message: stusb schematic
Other:
- sheet 0-10V Input ports: added VIN_3V3; removed none
- sheet MCU ports: added VIN_3V3; removed none
- note added: "da fixare nomenclature 3v3 ecc"
Changed lines of the file:
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@@
 	(generator_version "9.0")
 	(paper "A4")
+	(text "da fixare nomenclature 3v3 ecc"
+		(exclude_from_sim no)
+		(at 85.09 72.644 0)
+		(effects
+			(font
+				(size 1.27 1.27)
+				(thickness 0.254)
+				(bold yes)
+			)
+		)
+	)
+	(junction
+		(at 137.16 91.44)
+		(diameter 0)
+		(color 0 0 0 0)
+	)
 	(wire
 		(pts
@@
 	(wire
 		(pts
+			(xy 137.16 83.82) (xy 137.16 91.44)
+		)
+		(stroke
+			(width 0)
+			(type default)
+		)
+	)
+	(wire
+		(pts
 			(xy 156.21 104.14) (xy 144.78 104.14)
 		)
@@
 	(wire
 		(pts
+			(xy 105.41 96.52) (xy 105.41 91.44)
+		)
+		(stroke
+			(width 0)
+			(type default)
+		)
+	)
+	(wire
+		(pts
 			(xy 109.22 106.68) (xy 119.38 106.68)
+		)
+		(stroke
+			(width 0)
+			(type default)
+		)
+	)
+	(wire
+		(pts
+			(xy 137.16 91.44) (xy 137.16 96.52)
+		)
+		(stroke
+			(width 0)
+			(type default)
+		)
+	)
+	(wire
+		(pts
+			(xy 105.41 91.44) (xy 137.16 91.44)
 		)
 		(stroke
@@
 		)
 		(pin "VOUT_3V3" output
-			(at 124.46 83.82 270)
+			(at 137.16 83.82 270)
 			(effects
 				(font
@@
 			)
 		)
+		(pin "VIN_3V3" input
+			(at 137.16 96.52 90)
+			(effects
+				(font
+					(size 1.27 1.27)
+				)
+				(justify right)
+			)
+		)
 		(instances
 			(project "PCB"
@@
 			(effects
 				(font
+					(size 1.27 1.27)
+				)
+				(justify right)
+			)
+		)
+		(pin "VIN_3V3" input
+			(at 105.41 96.52 90)
+			(effects
+				(font
