File: PCB/mcu.kicad_sch (KiCad schematic)
At the start: 0 parts

Commit message: fix to 0-10V IN schematic, 0-10V OUT schematic
Other:
- note added: "PULL UP i2c su ESP"
- note added: "progtrm pin"
Changed lines of the file:
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@@
 	(generator_version "9.0")
 	(paper "A4")
+	(text "progtrm pin"
+		(exclude_from_sim no)
+		(at 46.99 51.562 0)
+		(effects
+			(font
+				(size 1.27 1.27)
+			)
+		)
+	)
+	(text "PULL UP i2c su ESP"
+		(exclude_from_sim no)
+		(at 48.768 57.658 0)
+		(effects
+			(font
+				(size 1.27 1.27)
+			)
+		)
+	)
 )

Commit message: minor fix, esp32 partial schematic
Parts:
- added C10: 1uF 50V X7R ±10% 0603, Capacitor_SMD:C_0603_1608Metric_Pad1.08x0.95mm_HandSolder, symbol Device:C
- added C8: 10uF 25V X5R ±20% 0603, Capacitor_SMD:C_0603_1608Metric_Pad1.08x0.95mm_HandSolder, symbol Device:C
- added C9: 100nF 50V X7R ±5% 0603, Capacitor_SMD:C_0603_1608Metric_Pad1.08x0.95mm_HandSolder, symbol Device:C
- added R10: 10K 5% 0603 1/10W, symbol Device:R
- added R11: 3K3 1% 0603 1/10W, symbol Device:R
- added U1: ESP32-C6-WROOM-1-N8, PCM_Espressif:ESP32-C6-WROOM-1, symbol PCM_Espressif:ESP32-C6-WROOM-1
Connections:
- new net +3V3: C8.1, C9.1, R10.2, R11.1, U1.2 (3V3)
- new net CHIP_PU: C10.2, R10.1, U1.3 (EN/CHIP_PU)
- new net GND: C10.1, C8.2, C9.2, U1.1 (GND), U1.28 (GND), U1.29 (GND)
- new net GPIO0: U1.8 (GPIO0/ADC1_CH0/XTAL_32K_P)
- new net GPIO1: U1.9 (GPIO1/ADC1_CH1/XTAL_32K_N)
- new net GPIO10: U1.11 (GPIO10)
- new net GPIO11: U1.12 (GPIO11)
- new net GPIO12: U1.13 (GPIO12/USB_D-)
- new net GPIO13: U1.14 (GPIO13/USB_D+)
- new net GPIO15: U1.23 (GPIO15)
- new net GPIO18: U1.16 (GPIO18)
- new net GPIO19: U1.17 (GPIO19)
- new net GPIO2: U1.27 (GPIO2/ADC1_CH2)
- new net GPIO20: U1.18 (GPIO20)
- new net GPIO21: U1.19 (GPIO21)
- new net GPIO22: U1.20 (GPIO22)
- new net GPIO23: U1.21 (GPIO23)
- new net GPIO3: U1.26 (GPIO3/ADC1_CH3)
- new net GPIO4: U1.4 (MTMS/GPIO4/ADC1_CH4)
- new net GPIO5: U1.5 (MTDI/GPIO5/ADC1_CH5)
- new net GPIO6: U1.6 (MTCK/GPIO6/ADC1_CH6)
- new net GPIO7: U1.7 (MTDO/GPIO7)
- new net GPIO8: R11.2, U1.10 (GPIO8)
- new net GPIO9: U1.15 (GPIO9)
- new net UART_RXD: U1.24 (U0RXD/GPIO17)
- new net UART_TXD: U1.25 (U0TXD/GPIO16)
Other:
- note added: "https://dl.espressif.com/dl/schematics/esp32-c6-devkitc-1-pcb-layout_v1.2.pdf"
- note added: "https://dl.espressif.com/dl/schematics/esp32-c6-devkitc-1-schematics_v1.4.pdf"
- note added: "https://documentation.espressif.com/esp32-c6-wroom-1_wroom-1u_datasheet_en.pdf"
- note added: "prevediamo quarzo? non so... nonm i convince...."

Commit message: esp32 various fix, 20to3v3 DCDC.
Parts:
- added C11: 100nF 50V X7R ±5% 0603, Capacitor_SMD:C_0603_1608Metric_Pad1.08x0.95mm_HandSolder, symbol Device:C
- added C12: 1uF 50V X7R ±10% 0603, Capacitor_SMD:C_0603_1608Metric_Pad1.08x0.95mm_HandSolder, symbol Device:C
- added D5: LED GREEN, Diode_SMD:D_0603_1608Metric_Pad1.05x0.95mm_HandSolder, symbol Device:LED
- added D6: LED BLUE, Diode_SMD:D_0603_1608Metric_Pad1.05x0.95mm_HandSolder, symbol Device:LED
- added FB2: 330Ohm@100MHz 0805, SamacSys_Parts:INDC2012X105N, symbol Device:FerriteBead
- added IC3: BC847BDW1T1G, SamacSys_Parts:SOT65P210X110-6N, symbol SamacSys_Parts:BC847BDW1T1G
- added J3: BM06B-GHS-TBT_LF__SN_, SamacSys_Parts:BM06BGHSTBTLFSN, symbol SamacSys_Parts:BM06B-GHS-TBT_LF__SN_
- added R12, R13: 10K 1% 0402 1/16W, Resistor_SMD:R_0402_1005Metric_Pad0.72x0.64mm_HandSolder, symbol Device:R
- added R14, R19, R22: 3K3 1% 0603 1/10W, Resistor_SMD:R_0603_1608Metric_Pad0.98x0.95mm_HandSolder, symbol Device:R
- added R15, R16, R17, R18: 100R 1% 0402 1/16W, Resistor_SMD:R_0402_1005Metric_Pad0.72x0.64mm_HandSolder, symbol Device:R
- added R20: 10K 5% 0603 1/10W, Resistor_SMD:R_0603_1608Metric_Pad0.98x0.95mm_HandSolder, symbol Device:R
- added R21: 330R 1% 0603, Resistor_SMD:R_0603_1608Metric_Pad0.98x0.95mm_HandSolder, symbol Device:R
- added R23: 220R 1% 0603, Resistor_SMD:R_0603_1608Metric_Pad0.98x0.95mm_HandSolder, symbol Device:R
- added S1: KSC221JLFS, SamacSys_Parts:KSC221JLFS, symbol SamacSys_Parts:KSC221JLFS
- added U2: ESD7004MUTAG, SamacSys_Parts:UDFN10_CASE_517BB, symbol SamacSys_Parts:ESD7004MUTAG
- R10, R11: footprint (none) -> Resistor_SMD:R_0603_1608Metric_Pad0.98x0.95mm_HandSolder
Connections:
- net +3V3: now also FB2.1, R14.1, R19.1, R20.2, R21.2, R23.2; no longer C8.1, C9.1, R10.2, R11.1, U1.2 (3V3)
- net GND: now also C11.2, C12.1, J3.1, J3.MP1, J3.MP2, S1.4 (NO_2), U2.3 (GND_1), U2.8 (GND_2)
- net GPIO22: now also D5.1 (K)
- net GPIO23: now also D6.1 (K)
- net GPIO4: now also R20.1, R22.1
- net GPIO9: now also IC3.6 (C2)
- net UART_RXD: now also R17.1
- net UART_TXD: now also R18.1
- net CHIP_PU renamed PG_IN
- net PG_IN: now also IC3.3 (C1)
- net GPIO1 renamed V_SENSE_IN
- net GPIO6 renamed SDA
- net SDA: now also R19.2
- net GPIO7 renamed SCL
- net SCL: now also R14.2
- new net: D5.2 (A), R21.1
- new net: C11.1, R22.2, S1.3 (COM_2)
- new net: R17.2, U2.2 (I/O_2)
- new net: IC3.2 (B2), R12.1
- new net: R18.2, U2.1 (I/O_1)
- new net: J3.2, U2.10 (N/C_4)
- new net: R16.2, U2.4 (I/O_3)
- new net: R15.2, U2.5 (I/O_4)
- new net: J3.5, U2.6 (N/C_1)
- new net: J3.4, U2.7 (N/C_2)
- new net: J3.3, U2.9 (N/C_3)
- new net: D6.2 (A), R23.1
- new net: IC3.5 (B1), R13.2
- new net +3V3_ESP: C12.2, C8.1, C9.1, FB2.2, R10.2, R11.1, U1.2 (3V3)
- new net DTR: IC3.1 (E2), R13.1, R16.1
- new net RTS: IC3.4 (E1), R12.2, R15.1
- no-connect marks 0 -> 3
Other:
- note added: "Auto program DTR RTS --> EN IO9 1 1 1 1 0 0 1 1 1 0 0 1 0 1 1 0"
- note added: "COSTLY!"
- note added: "LED"
- note added: "R10 to be removed after PG sequence is tested"
- note added: "perating life cycles: 300,000 cycles. Actuation force: 2 N (circa 200 gf). Operating temperature range: –40…+125 °C Square shape/size 6.2 x 6.2 mm, SMD mounting, IP67 sealed, low profile (3.5 mm height actuator), gold plated per high reliability."
- note added: "τ = R·C = 10 ms"
- note removed: "prevediamo quarzo? non so... nonm i convince...."
- moved on the sheet: C10, C8, C9, R10, R11, U1

Commit message: stusb schematic
Changed lines of the file:
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@@
 		)
 	)
+	(hierarchical_label "VIN_3V3"
+		(shape input)
+		(at 137.16 29.21 90)
+		(effects
+			(font
+				(size 1.27 1.27)
+				(thickness 0.254)
+				(bold yes)
+			)
+			(justify left)
+		)
+	)
 	(hierarchical_label "SDA"
 		(shape bidirectional)
@@
 					(unit 1)
 				)
+			)
+		)
+	)
+	(symbol
+		(lib_id "power:+3V3")
+		(at 137.16 29.21 180)
+		(unit 1)
+		(exclude_from_sim no)
+		(in_bom yes)
+		(on_board yes)
+		(dnp no)
+		(fields_autoplaced yes)
+		(property "Reference" "#PWR041"
+			(at 137.16 25.4 0)
+			(effects
+				(font
+					(size 1.27 1.27)
+				)
+				(hide yes)
+			)
+		)
+		(property "Value" "+3V3"
+			(at 137.16 34.29 0)
+			(effects
+				(font
+					(size 1.27 1.27)
+				)
+			)
+		)
+		(property "Footprint" ""
+			(at 137.16 29.21 0)
+			(effects
+				(font
+					(size 1.27 1.27)
+				)
+				(hide yes)
+			)
+		)
+		(property "Datasheet" ""
+			(at 137.16 29.21 0)
+			(effects
+				(font
+					(size 1.27 1.27)
+				)
+				(hide yes)
+			)
+		)
+		(property "Description" "Power symbol creates a global label with name \"+3V3\""
+			(at 137.16 29.21 0)
+			(effects
+				(font
+					(size 1.27 1.27)
+				)
+				(hide yes)
+			)
+		)
+		(pin "1"
+		)
+		(instances
+			(project "PCB"
+				(path "/6bd10cb8-11ca-4919-a8d8-88b44cd4cac7/872fc268-41bf-4357-ba67-172e8e148603"
+					(reference "#PWR041")
+					(unit 1)
+				)
