File: PCB/usb_pd.kicad_sch (KiCad schematic)
At the start: 0 parts

Commit message: stusb schematic
Parts:
- added C19, C20, C22, C24: 1uF 50V X7R ±10% 0603, Capacitor_SMD:C_0603_1608Metric_Pad1.08x0.95mm_HandSolder, symbol Device:C
- added C21: 4u7 50V 0805 X7R, Capacitor_SMD:C_0805_2012Metric_Pad1.18x1.45mm_HandSolder, symbol Device:C
- added C23: 100nF 50V X7R ±5% 0603, Capacitor_SMD:C_0603_1608Metric_Pad1.08x0.95mm_HandSolder, symbol Device:C
- added D10: BAT54JFILM, SOD2513X117N, symbol SamacSys_Parts:BAT54JFILM
- added D7, D9: ESDA25P35-1U1M, SamacSys_Parts:ESDA25P351U1M, symbol SamacSys_Parts:ESDA25P35-1U1M
- added D8: ESDA25W, SOT65P210X110-3N, symbol SamacSys_Parts:ESDA25W
- added J4: G-Switch GT-USB-7075A, USB_C:G-Switch GT-USB-7075A, symbol USB_C:G-Switch_GT-USB-7075A
- added J5: Conn_01x02_Socket, symbol Connector:Conn_01x02_Socket
- added Q1, Q2: STL6P3LLH6, STL8N10F7, symbol SamacSys_Parts:STL6P3LLH6
- added R28, R29, R30, R37: 10K 1% 0402 1/16W, Resistor_SMD:R_0402_1005Metric_Pad0.72x0.64mm_HandSolder, symbol Device:R
- added R31: 470R 5% 100mW 0603, symbol Device:R
- added R32: 1K 5% 100mW 0603, symbol Device:R
- added R33: 22K 5% 100mW 0603, symbol Device:R
- added R34: 100K 0603 5% 100mW, symbol Device:R
- added R35: 100R 0603 5% 100mW, symbol Device:R
- added R36: 1K 0603 1%, symbol Device:R
- added U3: STUSB4500QTR, Package_DFN_QFN:QFN-24-1EP_4x4mm_P0.5mm_EP2.7x2.7mm, symbol Interface_USB:STUSB4500QTR
Connections:
- new net: R29.1, U3.12 (ADDR0)
- new net: R28.1, U3.13 (ADDR1)
- new net: R33.2, U3.16 (VBUS_EN_SNK)
- new net: R32.2, U3.18 (VBUS_VS_DISCH)
- new net: D8.2 (CATHODE_2), J4.A5 (CC1), U3.2 (CC1)
- new net: C20.2, U3.21 (VREG_1V2)
- new net: C24.2, Q1.1 (S_1), Q1.2 (S_2), Q1.3 (S_3), Q2.1 (S_1), Q2.2 (S_2), Q2.3 (S_3), R34.1, U3.24 (VDD)
- new net: D8.1 (CATHODE_1), J4.B5 (CC2), U3.4 (CC2)
- new net: R36.1, U3.9 (DISCH)
- new net: Q1.4 (G), Q2.4 (G), R33.1, R34.2, R35.1
- new net: C22.2, D10.2 (K), R31.2, R32.1
- new net: C23.2, R35.2
- new net 2V7: C19.2, R28.2, R29.2, R37.2, U3.23 (VREG_2V7)
- new net GND: C19.1, C20.1, C21.2, C22.1, C24.1, D7.2 (A), D8.3 (ANODE), D9.2 (A), J4.1 (CASE), J4.A1 (GND), J4.A12 (GND), J4.B1 (GND), J4.B12 (GND), J5.1 (Pin_1), R30.1, U3.1 (CC1DB), U3.10 (GND), U3.22 (VSYS), U3.25 (GND), U3.5 (CC2DB)
- new net GPIO: R37.1, U3.15 (GPIO)
- new net RESET: R30.2, U3.6 (RESET)
- new net SCL: U3.7 (SCL)
- new net SDA: U3.19 (ALERT), U3.8 (SDA)
- new net VBUS: C21.1, D10.1 (A), D7.1 (K), J4.A4 (VBUS), J4.A9 (VBUS), J4.B4 (VBUS), J4.B9 (VBUS), Q2.5 (D_1), Q2.6 (D_2), Q2.7 (D_3), R31.1
- new net Vsnk: C23.1, D9.1 (K), J5.2 (Pin_2), Q1.5 (D_1), Q1.6 (D_2), Q1.7 (D_3), R36.2
- no-connect marks 0 -> 18
Other:
- note added: "G-Switch GT-USB-7075A"
- note added: "Powering a system under high charging profile only The STUSB4500 can be configured to allow the VBUS power path to be enabled by VBUS_EN_SNK pin only when a high power charging profile above 5 V has been negotiated (PDO2 or PDO3) with the source (see Section 3.3 Auto-run mode). This feature can be turned on thanks to NVM bit POWER_ONLY_ABOVE_5V (see Section 5 Start-up configuration). When the bit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"
- note added: "Warning: CC1DB and CC2DB must be connected to ground when dead battery mode is not supported."
- note added: "https://www.st.com/resource/en/data_brief/steval-isc005v1.pdf"
